File: board/tetrad.sch (EAGLE design)
At the start: 128 parts, among them Q1 FET-PCH-TO252, Q10 FET-NCH-SOT23, Q11 FET-NCH-SOT23, Q12 FET-NCH-SOT23, Q2 FET-NCH-SOT23, Q3 FET-NCH-SOT23, Q4 FET-NCH-SOT23, Q5 FET-NCH-SOT23, Q6 FET-NCH-SOT23, Q7 FET-NCH-SOT23, Q8 FET-NCH-SOT23, Q9 FET-NCH-SOT23, U1 IO-MCP23017ML, U2 RADIO-ESP32_DEVKIT, U3 R-78E5.0-1.0

Commit message: continued working on placement
Parts:
- added C17: 47u, holla:C-1206
Connections:
- removed net X_STEP_5V1: Q3.D
- removed net YA1: UY.A1
- removed net YA2: UY.A2
- removed net YB1: UY.B1
- removed net YB2: UY.B2
- new net N$37: R37.1, UY.M0
- new net N$38: R39.1, UY.M1
- new net N$39: R41.1, UY.M2
- new net N$40: R36.2, UY.A2, Y.6
- new net N$41: R42.2, UY.A1, Y.3
- new net N$42: R38.1, UY.B1, Y.2
- new net N$43: R40.1, UY.B2, Y.1
- new net N$44: Q12.D, R32.2
- net 24V0: now also C17.1, R42.1
- net 3V3: now also R37.2, R39.2, R41.2, UY.!RESET, UY.!SLEEP
- net 5V0: now also R40.2, UY.!FAULT; no longer A.1, Y.1, Z.1
- net GND: now also C17.2, UY.VMGND
- net N$21: now also Q3.D, R38.2; no longer Q12.D, R32.2, UX.STEP
- net N$5: no longer UX.DIR
- net N$6: now also Y.5
- net N$7: now also R36.1
- net X_DIR: now also UX.DIR
- net X_STEP: now also UX.STEP
- net Y_DIR: now also UY.DIR
- net Y_STEP: now also UY.STEP
Other:
- moved on the sheet: C10, C6, Q11, Q12, Q2, Q3, R19, R20, R26, R27, R32, R34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
