File: board/tetrad.brd (EAGLE design)
At the start: 122 x 122 mm, 128 parts, among them Q1 FET-PCH-TO252, Q10 FET-NCH-SOT23, Q11 FET-NCH-SOT23, Q12 FET-NCH-SOT23, Q2 FET-NCH-SOT23, Q3 FET-NCH-SOT23, Q4 FET-NCH-SOT23, Q5 FET-NCH-SOT23, Q6 FET-NCH-SOT23, Q7 FET-NCH-SOT23, Q8 FET-NCH-SOT23, Q9 FET-NCH-SOT23, U1 IO-MCP23017ML, U2 RADIO-ESP32_DEVKIT, U3 R-78E5.0-1.0

Commit message: continued working on placement
Parts:
- added C17: 47u, holla:C-1206
- moved C16 210.9 mm to (82.7, 20.8)
- moved R26 176.0 mm to (74.2, 15.6), turned to 180 degrees
- moved R27 173.7 mm to (74.2, 17.4), turned to 180 degrees
- moved Q11 30.2 mm to (103.0, 4.19)
- moved Q12 26.5 mm to (102.6, 9.53)
- moved J3V3 7.50 mm to (-73.3, 57.9)
- moved R30 4.10 mm to (78.5, 15.9), turned to 90 degrees
- moved R34 2.50 mm to (106.7, 4.19)
- moved RXM1 1.17 mm to (75.2, 5.33), flipped to the top, turned to 180 degrees
- moved RXM0 1.17 mm to (75.2, 3.56), flipped to the top, turned to 180 degrees
- moved RXM2 1.17 mm to (75.2, 7.11), flipped to the top, turned to 180 degrees
- moved R28 1.02 mm to (106.4, 12.7)
- moved R32 1.02 mm to (106.4, 9.53)
Connections:
- removed net X_STEP_5V1: Q3.3
- removed net YA1: UY.12, UY.12_
- removed net YA2: UY.11, UY.11_
- removed net YB1: UY.13, UY.13_
- removed net YB2: UY.14, UY.14_
- new net N$37: R37.1, UY.2, UY.2_
- new net N$38: R39.1, UY.3, UY.3_
- new net N$39: R41.1, UY.4, UY.4_
- new net N$40: R36.2, UY.11, UY.11_, Y.6, Y.6_
- new net N$41: R42.2, UY.12, UY.12_, Y.3, Y.3_
- new net N$42: R38.1, UY.13, UY.13_, Y.2, Y.2_
- new net N$43: R40.1, UY.14, UY.14_, Y.1, Y.1_
- new net N$44: Q12.3, R32.2
- net 24V0: now also C17.1, R42.1
- net 3V3: now also R37.2, R39.2, R41.2, UY.5, UY.5_, UY.6, UY.6_
- net 5V0: now also R40.2, UY.10, UY.10_; no longer A.1, A.1_, Y.1, Y.1_, Z.1, Z.1_
- net GND: now also C17.2, UY.15, UY.15_
- net N$21: now also Q3.3, R38.2; no longer Q12.3, R32.2, UX.7, UX.7_
- net N$5: no longer UX.8, UX.8_
- net N$6: now also Y.5, Y.5_
- net N$7: now also R36.1
- net VMGND: no longer UY.15, UY.15_
- net X_DIR: now also UX.8, UX.8_
- net X_STEP: now also UX.7, UX.7_
- net Y_DIR: now also UY.8, UY.8_
- net Y_STEP: now also UY.7, UY.7_
Routing:
- net X_STEP: track 0.00 -> 46.3 mm
- net X_DIR: track 0.00 -> 43.2 mm
- net N$5: track 38.3 -> 1.83 mm, vias 2 -> 0
- net N$21: track 33.8 -> 0.00 mm
- net X_LIMIT: track 0.00 -> 5.62 mm
- net N$33: track 8.70 -> 13.6 mm
- net N$34: track 11.9 -> 16.1 mm
- net N$35: track 15.8 -> 18.0 mm
- net N$2: track 51.2 -> 48.9 mm
- net N$44: track 0.00 -> 1.96 mm
- net N$25: track 54.3 -> 56.0 mm
- net N$31: track 36.6 -> 35.6 mm
- net N$30: track 32.1 -> 31.1 mm
- net 24V0: track 27.1 -> 28.1 mm
- net N$32: track 46.2 -> 45.5 mm

Commit message: XYZ tested  # Please enter the commit message for your changes. Lines starting
Parts:
- removed J2, J7: (no value), holla:MOLEX_430450614_430450615
- removed R43, R51, R53: DNP, holla:R-0603
- added C18, C19: DNP, holla:C-1206
- added ESTOP: (no value), holla:CONN-.100-2
- added R29: 10k, holla:R-0603
- C16, C17: value 47u -> DNP
Connections:
- removed net AA1: UA.12, UA.12_
- removed net AA2: UA.11, UA.11_
- removed net AB1: UA.13, UA.13_
- removed net AB2: UA.14, UA.14_
- removed net VMGND: UA.15, UA.15_, UZ.15, UZ.15_
- removed net X_STEP_5V2: Q5.3
- removed net X_STEP_5V3: Q7.3
- removed net ZA1: UZ.12, UZ.12_
- removed net ZA2: UZ.11, UZ.11_
- removed net ZB1: UZ.13, UZ.13_
- removed net ZB2: UZ.14, UZ.14_
- new net ESTOP: ESTOP.2, R29.1, UA.1, UA.1_, UX.1, UX.1_, UY.1, UY.1_, UZ.1, UZ.1_
- new net N$36: Q6.3, R50.1
- new net N$45: R55.1, UA.2, UA.2_
- new net N$46: R45.1, UZ.2, UZ.2_
- new net N$47: R47.1, UZ.3, UZ.3_
- new net N$48: R49.1, UZ.4, UZ.4_
- new net N$49: R57.1, UA.3, UA.3_
- new net N$50: Q5.3, R44.1
- new net N$51: R46.2, UZ.11, UZ.11_, Z.6, Z.6_
- new net N$52: Q4.3, R46.1
- new net N$53: R44.2, UZ.13, UZ.13_, Z.2, Z.2_
- new net N$54: R54.2, UZ.12, UZ.12_, Z.3, Z.3_
- new net N$55: R59.1, UA.4, UA.4_
- new net N$56: R52.1, UZ.14, UZ.14_, Z.1, Z.1_
- new net N$58: A.6, A.6_, R50.2, UA.11, UA.11_
- new net N$59: A.3, A.3_, R58.2, UA.12, UA.12_
- new net N$60: A.2, A.2_, R48.2, UA.13, UA.13_
- net 24V0: now also C18.1, C19.1, R54.1, R58.1
- net 3V3: now also R29.2, R45.2, R47.2, R49.2, R55.2, R57.2, R59.2, UA.5, UA.5_, UA.6, UA.6_, UZ.5, UZ.5_, UZ.6, UZ.6_
- net 5V0: now also R52.2, R56.2, UA.10, UA.10_, UZ.10, UZ.10_
- net A_DIR: now also UA.8, UA.8_
- net A_STEP: now also UA.7, UA.7_
- net GND: now also C18.2, C19.2, ESTOP.1, UA.15, UA.15_, UZ.15, UZ.15_
- net N$10: now also A.5, A.5_
- net N$11: now also Q7.3, R48.1; no longer Q6.3
- net N$21: now also R38.1; no longer R38.2
- net N$42: now also R38.2; no longer R38.1
- net N$8: now also Z.5, Z.5_
- net N$9: now also A.1, A.1_, R56.1, UA.14, UA.14_; no longer Q4.3
- net Z_DIR: now also UZ.8, UZ.8_
- net Z_STEP: now also UZ.7, UZ.7_

Commit message: checked out the spindle hardware started to simplify the motor part of schematic
Parts:
- removed R32, R34: 0, holla:R-0603
- removed RXM0, RXM1, RXM2: DNP, holla:R-0603
- added F1: 10A, holla:3557-2
- added J2: (no value), holla:CONN-.100-4
- added J3: (no value), holla:AMPHENOL_95278-101A06LF
- R26: value 10k -> 1k
- R28, R30: value 0 -> 1k
- moved R28 320.1 mm to (-126.5, -206.9), turned to 0 degrees
- moved R30 306.4 mm to (-126.5, -211.8), turned to 0 degrees
Connections:
- removed net N$30: R28.1, UX.12, UX.12_, X.3, X.3_
- removed net N$32: R30.1, UX.14, UX.14_, X.1, X.1_
- removed net N$44: Q12.3, R32.2
- new net N$57: F1.2@1, F1.2@2, Q1.3
- new net N$62: J2.2, UX.12, UX.12_
- new net N$63: J2.3, UX.13, UX.13_
- new net N$64: J2.4, UX.14, UX.14_
- net 24V0: now also X.3, X.3_; no longer R28.2
- net 3V3: no longer RXM0.2, RXM1.2, RXM2.2, UX.5, UX.5_, UX.6, UX.6_
- net 5V0: now also J3.2, J3.4, J3.6, R28.1, R30.1, UX.5, UX.5_, UX.6, UX.6_, X.1, X.1_; no longer R30.2
- net N$1: now also F1.1@1, F1.1@2; no longer Q1.3
- net N$25: now also J2.1; no longer R34.2, X.6, X.6_
- net N$31: now also Q12.3, R28.2; no longer R32.1, UX.13, UX.13_
- net N$33: now also J3.5; no longer RXM0.1
- net N$34: now also J3.3; no longer RXM1.1
- net N$35: now also J3.1; no longer RXM2.1
- net N$5: now also R30.2, X.6, X.6_; no longer R34.1
Routing:
- net N$32: track 45.5 -> 0.00 mm, vias 1 -> 0
- net 5V0: track 0.00 -> 42.2 mm, vias 0 -> 1
- net N$30: track 31.1 -> 0.00 mm
- net N$25: track 56.0 -> 33.1 mm, vias 1 -> 0
- net N$31: track 35.6 -> 28.8 mm
- net 24V0: track 28.1 -> 25.3 mm
- net N$33: track 13.6 -> 11.3 mm
- net N$34: track 16.1 -> 13.9 mm
- net N$44: track 1.96 -> 0.00 mm
- net N$5: track 1.83 -> 0.00 mm
- net N$35: track 18.0 -> 16.5 mm

Commit message: schematic   updated alot   moving to bud PN-1325-DGMB enclosure initial add for others
Parts:
- removed 3V3: (no value), holla:TPTHRU
- removed A, X, Y, Z: (no value), holla:MOLEX_430450614_430450615
- removed C19: DNP, holla:C-1206
- removed DISPLAY: (no value), holla:1X08
- removed J3: (no value), holla:AMPHENOL_95278-101A06LF
- removed Q11, Q12, Q6, Q7: FET-NCH-SOT23, holla:SOT23-3
- removed UA, UX, UY, UZ: (no value), holla:IC_DRV8825_CARRIER_TH_SMD
- added AALT, XALT, YALT, ZALT: (no value), holla:MOLEX_430450614_430450615
- added ADRIVER, XDRIVER, YDRIVER, ZDRIVER: (no value), holla:IC_DRV8825_CARRIER_TH_SMD
- added ALIMIT, XLIMIT, YLIMIT, ZLIMIT: (no value), holla:CONN-.100-2
- added AMOTOR, XMOTOR, YMOTOR, ZMOTOR: (no value), holla:CONN-.100-4
- added AMSEL, XMSEL, YMSEL, ZMSEL: (no value), holla:AMPHENOL_95278-101A06LF
- added AUDIO: (no value), holla:TPTHRU
- added C20: .1u, holla:C-0603
- added D3, D4, D5, D6: (no value), holla:D-SOD523
- added D7, D8, D9: DNP, holla:D-SOD523
- added IC1: (no value), holla:SO20W
- added J16: (no value), holla:2X5-SHROUDED
- added R31, R51, R60, R61: DNP, holla:R-0603
- added R32, R33, R34, R35: 0, holla:R-0603
- added R43, R53: 1k, holla:R-0603
- added U13: (no value), holla:FCI_10051922-2010ELF
- C1, C9: value 1u -> .1u
- C13: value 1u -> DNP; device holla:C-0603 -> holla:C-1206
- C17: value DNP -> .1u; device holla:C-1206 -> holla:C-0603
- C6: value .1u -> DNP; device holla:C-0603 -> holla:C-1206
- J2: device holla:CONN-.100-4 -> holla:CONN-3.81MM-KF2EDG-6
- Q2, Q3, Q4, Q5: value FET-NCH-SOT23 -> FET-NCH-TO252; device holla:SOT23-3 -> holla:TO252
- R18: value 10k -> 100
- R19, R9: value 100 -> 1k
- R20: value 10k -> DNP
- R21, R22, R8: value 100 -> 0
- R23: value 10k -> 0
- R28: value 1k -> 100
- R30: value 1k -> DNP
- R36, R40, R44, R50, R54: value 0 -> DNP
- R42, R52: value 0 -> 100
- R45, R47, R55, R57: value DNP -> 0
- moved R28 334.0 mm to (170.0, -53.0), turned to 90 degrees
- moved J2 326.6 mm to (193.0, -85.0), turned to 90 degrees
- moved C9 303.0 mm to (180.0, -53.0), turned to 90 degrees
- moved Q2 277.9 mm to (174.0, -63.0)
- moved Q3 277.2 mm to (174.0, -75.0)
- moved Q5 270.4 mm to (174.0, -99.0)
- moved Q4 269.9 mm to (174.0, -87.0)
- moved C1 254.4 mm to (175.0, -53.0)
- moved J1 217.0 mm to (181.0, 80.0), turned to 90 degrees
- moved R52 208.5 mm to (79.0, -111.0), turned to 90 degrees
- moved R58 207.2 mm to (79.0, -87.0), turned to 90 degrees
- moved R55 207.2 mm to (79.0, -99.0), turned to 90 degrees
- moved R59 203.4 mm to (79.0, -83.0), turned to 90 degrees
- moved R56 203.0 mm to (79.0, -95.0), turned to 90 degrees
- moved R54 199.7 mm to (79.0, -103.0), turned to 90 degrees
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Connections:
- new net A_DIR': ADRIVER.8, ADRIVER.8_, IC1.11, R60.1
- new net A_STEP': ADRIVER.7, ADRIVER.7_, IC1.12, R61.1
- new net N$108: R8.2, U13.3, U13.4
- new net N$30: D5.A, J2.3, Q4.3
- new net N$32: D4.A, J2.4, Q3.3
- new net N$44: D3.A, J2.5, Q2.3
- new net N$61: ADRIVER.3, ADRIVER.3_, AMSEL.3
- new net N$65: ADRIVER.12, ADRIVER.12_, AMOTOR.2, R56.2
- new net N$66: ADRIVER.13, ADRIVER.13_, AMOTOR.3, R57.2
- new net N$67: ADRIVER.14, ADRIVER.14_, AMOTOR.4, R58.2
- new net N$68: AALT.5, AALT.5_, ALIMIT.2, R52.1, R53.1
- new net N$69: AALT.6, AALT.6_, R58.1, R60.2
- new net N$70: AALT.1, AALT.1_, R55.1, R59.2
- new net N$71: AALT.3, AALT.3_, R54.1, R57.1
- new net X_DIR': IC1.17, R36.1, XDRIVER.8, XDRIVER.8_
- new net X_STEP': IC1.18, R22.1, R33.1, R37.1, R37.2, R41.2, R46.1, R51.2, XALT.2, XALT.2_, XDRIVER.7, XDRIVER.7_, YALT.2, YALT.2_, ZALT.2, ZALT.2_
- new net X_STEP'1: AALT.2, AALT.2_, R56.1, R61.2
- new net Y_DIR': IC1.15, R40.1, YDRIVER.8, YDRIVER.8_
- new net Y_STEP': IC1.16, R41.1, YDRIVER.7, YDRIVER.7_
- new net Z_DIR': IC1.13, R50.1, ZDRIVER.8, ZDRIVER.8_
- new net Z_STEP': IC1.14, R51.1, ZDRIVER.7, ZDRIVER.7_
- net 24V0: now also ADRIVER.16, ADRIVER.16_, C13.1, C6.1, D3.C, D4.C, D5.C, D6.C, D7.C, D8.C, D9.C, J2.6, R20.2, R30.2, R44.2, R54.2, XDRIVER.16, XDRIVER.16_, YDRIVER.16, YDRIVER.16_, ZDRIVER.16, ZDRIVER.16_; no longer C17.1, C19.1, R42.1, R54.1, R58.1, UA.16, UA.16_, UX.16, UX.16_, UY.16, UY.16_, UZ.16, UZ.16_, X.3, X.3_
- net 3V3: now also C1.1, C9.1, J16.1, R19.2, R43.2, R53.2, R8.1, R9.2, U13.20, U13.5; no longer 3V3.1, C1.2, C13.2, C9.2, R18.2, R20.2, R23.2, R37.2, R39.2, R41.2, R45.2, R47.2, R49.2, R55.2, R57.2, R59.2, UA.5, UA.5_, UA.6, UA.6_, UY.5, UY.5_, UY.6, UY.6_, UZ.5, UZ.5_, UZ.6, UZ.6_
- net 5V0: now also ADRIVER.10, ADRIVER.10_, ADRIVER.5, ADRIVER.5_, ADRIVER.6, ADRIVER.6_, AMSEL.2, AMSEL.4, AMSEL.6, C20.1, IC1.20, R31.1, R39.1, R49.1, R59.1, XDRIVER.10, XDRIVER.10_, XDRIVER.5, XDRIVER.5_, XDRIVER.6, XDRIVER.6_, XMSEL.2, XMSEL.4, XMSEL.6, YDRIVER.10, YDRIVER.10_, YDRIVER.5, YDRIVER.5_, YDRIVER.6, YDRIVER.6_, YMSEL.2, YMSEL.4, YMSEL.6, ZDRIVER.10, ZDRIVER.10_, ZDRIVER.5, ZDRIVER.5_, ZDRIVER.6, ZDRIVER.6_, ZMSEL.2, ZMSEL.4, ZMSEL.6; no longer DISPLAY.2, J3.2, J3.4, J3.6, R28.1, R30.1, R40.2, R52.2, R56.2, UA.10, UA.10_, UX.10, UX.10_, UX.5, UX.5_, UX.6, UX.6_, UY.10, UY.10_, UZ.10, UZ.10_, X.1, X.1_
- net AUDIO: now also AUDIO.1, J16.9, U13.11
- net A_DIR: now also IC1.9; no longer Q6.1, UA.8, UA.8_
- net A_LIMIT: no longer C11.1, R22.2
- net A_STEP: now also IC1.8; no longer Q7.1, UA.7, UA.7_
- net CS_DISPLAY: now also J16.6, U13.15
- net DISPLAY_CS: no longer DISPLAY.7
- net DISPLAY_DC: no longer DISPLAY.6
- net ESTOP: now also ADRIVER.1, ADRIVER.1_, R28.1, XDRIVER.1, XDRIVER.1_, YDRIVER.1, YDRIVER.1_, ZDRIVER.1, ZDRIVER.1_; no longer UA.1, UA.1_, UX.1, UX.1_, UY.1, UY.1_, UZ.1, UZ.1_
- net GND: now also AALT.4, AALT.4_, ADRIVER.15, ADRIVER.15_, ADRIVER.9, ADRIVER.9_, ALIMIT.1, C1.2, C13.2, C20.2, C9.2, IC1.10, IC1.19, J16.10, J16.2, J2.1, U13.1, U13.19, U13.2, U13.6, U13.G1, U13.G2, XALT.4, XALT.4_, XDRIVER.15, XDRIVER.15_, XDRIVER.9, XDRIVER.9_, XLIMIT.1, YALT.4, YALT.4_, YDRIVER.15, YDRIVER.15_, YDRIVER.9, YDRIVER.9_, YLIMIT.1, ZALT.4, ZALT.4_, ZDRIVER.15, ZDRIVER.15_, ZDRIVER.9, ZDRIVER.9_, ZLIMIT.1; no longer A.4, A.4_, C1.1, C13.1, C19.2, C9.1, DISPLAY.1, Q11.2, Q12.2, Q6.2, Q7.2, UA.15, UA.15_, UA.9, UA.9_, UX.15, UX.15_, UX.9, UX.9_, UY.15, UY.15_, UY.9, UY.9_, UZ.15, UZ.15_, UZ.9, UZ.9_, X.4, X.4_, Y.4, Y.4_, Z.4, Z.4_
- net INT_DISPLAY: now also J16.7, U13.14
- net MISO: now also J16.4, U13.17
- net MOSI: now also J16.5, U13.16; no longer R8.2
- net N$10: now also R22.2, YDRIVER.12, YDRIVER.12_, YMOTOR.2; no longer A.5, A.5_, R22.1, R23.1
- net N$11: now also R23.2, YDRIVER.13, YDRIVER.13_, YMOTOR.3; no longer Q7.3, R48.1
- net N$13: now also D7.A
- net N$14: now also D9.A
- net N$18: now also R1.1
- net N$19: now also R7.1
- net N$2: now also R30.1, R34.1, XALT.3, XALT.3_; no longer R26.1, R27.1, X.5, X.5_
- net N$20: now also D6.A, J2.2, Q5.3; no longer DISPLAY.8
- net N$21: now also R38.2, YDRIVER.14, YDRIVER.14_, YMOTOR.4; no longer Q3.3, R38.1
- net N$25: now also R32.2, XDRIVER.11, XDRIVER.11_, XMOTOR.1; no longer J2.1, UX.11, UX.11_
- net N$3: now also IC1.1; no longer DISPLAY.3
- net N$31: now also R18.1, R19.1, YALT.5, YALT.5_, YLIMIT.2; no longer Q12.3, R28.2, X.2, X.2_
- net N$33: now also XDRIVER.2, XDRIVER.2_, XMSEL.5; no longer J3.5, UX.2, UX.2_
- net N$34: now also XDRIVER.3, XDRIVER.3_, XMSEL.3; no longer J3.3, UX.3, UX.3_
- net N$35: now also XDRIVER.4, XDRIVER.4_, XMSEL.1; no longer J3.1, UX.4, UX.4_
- net N$36: now also R38.1, R40.2, YALT.6, YALT.6_; no longer Q6.3, R50.1
- net N$37: now also R21.1, R39.2, YALT.1, YALT.1_; no longer R37.1, UY.2, UY.2_
- net N$38: now also R20.1, R23.1, YALT.3, YALT.3_; no longer R39.1, UY.3, UY.3_
- net N$39: now also R45.2, ZDRIVER.11, ZDRIVER.11_, ZMOTOR.1; no longer R41.1, UY.4, UY.4_
- net N$4: now also R28.2; no longer DISPLAY.4, R8.1
- net N$40: now also ZDRIVER.2, ZDRIVER.2_, ZMSEL.5; no longer R36.2, UY.11, UY.11_, Y.6, Y.6_
- net N$41: now also ZDRIVER.3, ZDRIVER.3_, ZMSEL.3; no longer R42.2, UY.12, UY.12_, Y.3, Y.3_
- net N$42: now also ZDRIVER.4, ZDRIVER.4_, ZMSEL.1; no longer R38.2, UY.13, UY.13_, Y.2, Y.2_
- net N$43: now also R46.2, ZDRIVER.12, ZDRIVER.12_, ZMOTOR.2; no longer R40.1, UY.14, UY.14_, Y.1, Y.1_
- net N$45: now also R47.2, ZDRIVER.13, ZDRIVER.13_, ZMOTOR.3; no longer R55.1, UA.2, UA.2_
- net N$46: now also R48.2, ZDRIVER.14, ZDRIVER.14_, ZMOTOR.4; no longer R45.1, UZ.2, UZ.2_
- net N$47: now also R42.1, R43.1, ZALT.5, ZALT.5_, ZLIMIT.2; no longer R47.1, UZ.3, UZ.3_
- net N$48: now also R48.1, R50.2, ZALT.6, ZALT.6_; no longer R49.1, UZ.4, UZ.4_
- net N$49: now also R45.1, R49.2, ZALT.1, ZALT.1_; no longer R57.1, UA.3, UA.3_
- net N$5: now also R31.2, R32.1, XALT.1, XALT.1_; no longer Q11.3, R30.2, X.6, X.6_
- net N$50: now also R47.1, ZALT.3, ZALT.3_; no longer Q5.3
- net N$51: now also ADRIVER.11, ADRIVER.11_, AMOTOR.1, R55.2; no longer R46.2, UZ.11, UZ.11_, Z.6, Z.6_
- net N$52: now also Q2.1, U1.1; no longer Q4.3, R46.1
- net N$53: now also Q3.1, U1.2; no longer R44.2, UZ.13, UZ.13_, Z.2, Z.2_
- net N$54: now also Q4.1, U1.3; no longer R54.2, UZ.12, UZ.12_, Z.3, Z.3_
- net N$55: now also Q5.1, U1.4; no longer R59.1, UA.4, UA.4_
- net N$56: now also R35.2, XDRIVER.14, XDRIVER.14_, XMOTOR.4; no longer R52.1, UZ.14, UZ.14_, Z.1, Z.1_
- net N$58: now also R26.1, R27.1, XALT.5, XALT.5_, XLIMIT.2; no longer A.6, A.6_, R50.2, UA.11, UA.11_
- net N$59: now also ADRIVER.2, ADRIVER.2_, AMSEL.5; no longer A.3, A.3_, R58.2, UA.12, UA.12_
- net N$6: now also R21.2, YDRIVER.11, YDRIVER.11_, YMOTOR.1; no longer R19.1, R20.1, Y.5, Y.5_
- net N$60: now also R35.1, R36.2, XALT.6, XALT.6_; no longer A.2, A.2_, R48.2, UA.13, UA.13_
- net N$62: now also R33.2, XDRIVER.12, XDRIVER.12_, XMOTOR.2; no longer J2.2, UX.12, UX.12_
- net N$63: now also R34.2, XDRIVER.13, XDRIVER.13_, XMOTOR.3; no longer J2.3, UX.13, UX.13_
- net N$64: now also ADRIVER.4, ADRIVER.4_, AMSEL.1; no longer J2.4, UX.14, UX.14_
- net N$7: now also YDRIVER.2, YDRIVER.2_, YMSEL.5; no longer Q2.3, R36.1
- net N$8: now also YDRIVER.3, YDRIVER.3_, YMSEL.3; no longer R18.1, R21.1, Z.5, Z.5_
- net N$9: now also YDRIVER.4, YDRIVER.4_, YMSEL.1; no longer A.1, A.1_, R56.1, UA.14, UA.14_
- net PD_DISPLAY: now also J16.8, U13.13
- net RESET: no longer DISPLAY.5
- net SCK: now also J16.3, U13.18; no longer R9.2
- net SCL: no longer R1.1
- net SDA: no longer R7.1
- net X_DIR: now also IC1.3; no longer Q11.1, UX.8, UX.8_
- net X_LIMIT: now also C11.1, C17.1, C4.1, R18.2, R42.2, R52.2
- net X_STEP: now also IC1.2; no longer Q12.1, UX.7, UX.7_
- net X_STEP_5V4: now also D8.A
- net Y_DIR: now also IC1.5; no longer Q2.1, UY.8, UY.8_
- net Y_LIMIT: no longer C6.1, R19.2
- net Y_STEP: now also IC1.4; no longer Q3.1, UY.7, UY.7_
- net Z_DIR: now also IC1.7; no longer Q4.1, UZ.8, UZ.8_
- net Z_LIMIT: no longer C4.1, R21.2
- net Z_STEP: now also IC1.6; no longer Q5.1, UZ.7, UZ.7_
Routing:
- net N$2: track 48.9 -> 0.00 mm
- net X_STEP: track 46.3 -> 0.00 mm
- net X_DIR: track 43.2 -> 0.00 mm
- net 5V0: track 42.2 -> 0.00 mm, vias 1 -> 0
- net N$25: track 33.1 -> 0.00 mm
- net N$31: track 28.8 -> 0.00 mm
- net 24V0: track 25.3 -> 0.00 mm
- net N$35: track 16.5 -> 0.00 mm
- net N$34: track 13.9 -> 0.00 mm
- net N$33: track 11.3 -> 0.00 mm
- net X_LIMIT: track 5.62 -> 0.00 mm
Other:
- board size 122 x 122 mm -> 197 x 98 mm
