File: release/v1.0/hexad.sch (EAGLE design)
At the start: 128 parts, among them Q1 FET-PCH-TO252, Q10 FET-NCH-SOT23, Q11 FET-NCH-SOT23, Q12 FET-NCH-SOT23, Q2 FET-NCH-SOT23, Q3 FET-NCH-SOT23, Q4 FET-NCH-SOT23, Q5 FET-NCH-SOT23, Q6 FET-NCH-SOT23, Q7 FET-NCH-SOT23, Q8 FET-NCH-SOT23, Q9 FET-NCH-SOT23, U1 IO-MCP23017ML, U2 RADIO-ESP32_DEVKIT, U3 R-78E5.0-1.0

Commit message: XYZ tested  # Please enter the commit message for your changes. Lines starting
Parts:
- removed C16, C17, C18, C19: DNP, holla:C-1206
- removed ESTOP: (no value), holla:CONN-02-.100-VERT-HEADER
- removed J17: (no value), holla:CONN-20-2-84952-0
- removed R28, R30, R32, R34, R36, R38, R40, R42, R44, R46, R48, R50, R52, R54, R56, R58: 0, holla:R-0603
- removed R29: 10k, holla:R-0603
- removed R37, R39, R41, R45, R47, R49, R55, R57, R59, RXM0, RXM1, RXM2: DNP, holla:R-0603
- removed UA, UX, UY, UZ: (no value), holla:BOARD-DRV8825-CARRIER-TH-SMD
- A, X, Y, Z: device holla:CONN-03X2-MICROFIT-TH-SMD -> holla:CONN-06-.100-VERT-HEADER
- Q1: value FET-PCH-TO252 -> 40V
- Q10, Q11, Q12, Q2, Q3, Q4, Q5, Q6, Q7, Q8, Q9: value FET-NCH-SOT23 -> (none)
- R1, R7: value 1k -> 2k
- U1: value IO-MCP23017ML -> (none); device holla:IO-MCP23017ML -> holla:IO-MCP23017SO
Connections:
- removed net AUDIO: J17.9
- removed net CS_DISPLAY: J17.6
- removed net ESTOP: ESTOP.2, R29.1, UA.!ENABLE, UX.!ENABLE, UY.!ENABLE, UZ.!ENABLE
- removed net INT_DISPLAY: J17.7
- removed net N$21: Q3.D, R38.1
- removed net N$25: R34.2, UX.A2, X.6
- removed net N$30: R28.1, UX.A1, X.3
- removed net N$31: R32.1, UX.B1, X.2
- removed net N$32: R30.1, UX.B2, X.1
- removed net N$33: RXM0.1, UX.M0
- removed net N$34: RXM1.1, UX.M1
- removed net N$35: RXM2.1, UX.M2
- removed net N$36: Q6.D, R50.1
- removed net N$37: R37.1, UY.M0
- removed net N$38: R39.1, UY.M1
- removed net N$39: R41.1, UY.M2
- removed net N$40: R36.2, UY.A2, Y.6
- removed net N$41: R42.2, UY.A1, Y.3
- removed net N$42: R38.2, UY.B1, Y.2
- removed net N$43: R40.1, UY.B2, Y.1
- removed net N$44: Q12.D, R32.2
- removed net N$45: R55.1, UA.M0
- removed net N$46: R45.1, UZ.M0
- removed net N$47: R47.1, UZ.M1
- removed net N$48: R49.1, UZ.M2
- removed net N$49: R57.1, UA.M1
- removed net N$50: Q5.D, R44.1
- removed net N$51: R46.2, UZ.A2, Z.6
- removed net N$52: Q4.D, R46.1
- removed net N$53: R44.2, UZ.B1, Z.2
- removed net N$54: R54.2, UZ.A1, Z.3
- removed net N$55: R59.1, UA.M2
- removed net N$56: R52.1, UZ.B2, Z.1
- removed net N$58: A.6, R50.2, UA.A2
- removed net N$59: A.3, R58.2, UA.A1
- removed net N$60: A.2, R48.2, UA.B1
- removed net PD_DISPLAY: J17.8
- new net X_STEP_5V0: Q12.D, X.3
- new net X_STEP_5V1: Q3.D, Y.3
- new net X_STEP_5V2: Q5.D, Z.3
- new net X_STEP_5V3: A.3, Q7.D
- net 24V0: now also A.6, X.6, Y.6, Z.6; no longer C16.1, C17.1, C18.1, C19.1, R28.2, R42.1, R54.1, R58.1, UA.VMOTOR, UX.VMOTOR, UY.VMOTOR, UZ.VMOTOR
- net 3V3: no longer J17.1, J17.17, J17.18, R29.2, R37.2, R39.2, R41.2, R45.2, R47.2, R49.2, R55.2, R57.2, R59.2, RXM0.2, RXM1.2, RXM2.2, UA.!RESET, UA.!SLEEP, UX.!RESET, UX.!SLEEP, UY.!RESET, UY.!SLEEP, UZ.!RESET, UZ.!SLEEP
- net 5V0: now also A.5, X.5, Y.5, Z.5; no longer R30.2, R40.2, R52.2, R56.2, UA.!FAULT, UX.!FAULT, UY.!FAULT, UZ.!FAULT
- net A_DIR: now also U2.D2; no longer U2.T2/D02, UA.DIR
- net A_LIMIT: now also U2.D4; no longer U2.T0/D04
- net A_STEP: now also U2.D15; no longer U2.T3/D15, UA.STEP
- net CS_SD: now also U2.D34; no longer U2.D25/DAC1
- net CYCLE_START: now also U2.VN/AD3/D39; no longer U2.D39/VN
- net FEED_HOLD: now also U2.VP/AD0/D36; no longer U2.D36/VP
- net GND: now also A.1, X.1, Y.1, Z.1; no longer A.4, C16.2, C17.2, C18.2, C19.2, ESTOP.1, J17.19, J17.2, J17.20, UA.GND, UA.VMGND, UX.GND, UX.VMGND, UY.GND, UY.VMGND, UZ.GND, UZ.VMGND, X.4, Y.4, Z.4
- net MISO: now also U2.D19; no longer J17.4, U2.MISO/D19
- net MOSI: now also U2.D23; no longer J17.5, U2.MOSI/D23
- net N$10: now also A.4; no longer A.5
- net N$11: now also A.2, Q6.D; no longer Q7.D, R48.1
- net N$2: now also X.4; no longer X.5
- net N$5: now also X.2; no longer R34.1
- net N$6: now also Y.4; no longer Y.5
- net N$7: now also Y.2; no longer R36.1
- net N$8: now also Z.4; no longer Z.5
- net N$9: now also Q4.D, Z.2; no longer A.1, R56.1, UA.B2
- net SCK: now also U2.D18; no longer J17.3, U2.SCLK/D18
- net SCL: now also U2.D22; no longer U2.SCL/D22
- net SDA: now also U2.D21; no longer U2.SDA/D21
- net SPINDLE_DIR: now also U2.D16/RX2; no longer U2.RX2/D16
- net SPINDLE_ENABLE: now also U2.D5; no longer U2.SS/D05
- net SPINDLE_PWM: now also U2.D17/TX2; no longer U2.TX2/D17
- net X_DIR: now also U2.D12; no longer U2.D12/T5, UX.DIR
- net X_LIMIT: now also U2.D14; no longer U2.D14/T6
- net X_STEP: now also U2.D13; no longer U2.D13/T4, UX.STEP
- net Y_DIR: now also U2.D26; no longer U2.D26/DAC2, UY.DIR
- net Y_LIMIT: now also U2.D25; no longer U2.D34_IN_ONLY
- net Y_STEP: now also U2.D27; no longer U2.D27/T7, UY.STEP
- net Z_DIR: now also U2.D32; no longer U2.D32/T9, UZ.DIR
- net Z_LIMIT: now also U2.D35; no longer U2.D35_IN_ONLY
- net Z_STEP: now also U2.D33; no longer U2.D33/T8, UZ.STEP
Other:
- note removed: "40V"
- note removed: "47u"
- note removed: "V1.1"
- note removed: "todo add EVE2 display connector CS_SD is on an input only pin, fix this replace esp32 with new lib part, reroute check audio pin on FFC connector https://randomnerdtutorials.com/esp32-pinout-reference-gpios/ check if D14 and D15 PWM out on startup add 0430450612 headers add drv8825 board headers switch 23017 to qfn"
